File: PionController/_autosave-PionController.kicad_pcb (KiCad board)
At the start: 2 copper layers, 1 part, among them U1 STM32H743VITx

Commit message: Schematic_ready
Parts:
- added C1: 10uF, Capacitor_SMD:C_1210_3225Metric, F.Cu at (101.0, 66.2)
- added C10: 2.2uF, Capacitor_SMD:C_0603_1608Metric, F.Cu at (102.0, 80.8)
- added C11: 10uF, Capacitor_SMD:C_1210_3225Metric, F.Cu at (116.0, 57.5)
- added C12: 2.2uF, Capacitor_SMD:C_0603_1608Metric, F.Cu at (103.2, 123.5)
- added C13: 2.2uF, Capacitor_SMD:C_0603_1608Metric, F.Cu at (103.2, 126.0)
- added C14: 100nF, Capacitor_SMD:C_0603_1608Metric, F.Cu at (118.5, 72.5)
- added C15: 100nF, Capacitor_SMD:C_0603_1608Metric, F.Cu at (123.2, 83.5)
- added C16: 100nF, Capacitor_SMD:C_0603_1608Metric, F.Cu at (135.0, 84.0)
- added C17: 100nF, Capacitor_SMD:C_0603_1608Metric, F.Cu at (139.0, 67.5)
- added C18: 100nF, Capacitor_SMD:C_0603_1608Metric, F.Cu at (123.3, 63.5)
- added C19: 100nF, Capacitor_SMD:C_0603_1608Metric, F.Cu at (118.5, 70.0)
- added C2: 10uF, Capacitor_SMD:C_1210_3225Metric, F.Cu at (95.7, 67.8)
- added C20: 2.2uF, Capacitor_SMD:C_0603_1608Metric, F.Cu at (118.2, 86.3)
- added C21: 2.2uF, Capacitor_SMD:C_0603_1608Metric, F.Cu at (117.5, 81.2)
- added C22: 100nF, Capacitor_SMD:C_0603_1608Metric, F.Cu at (120.8, 86.2)
- added C23: 100nF, Capacitor_SMD:C_0603_1608Metric, F.Cu at (113.5, 81.2)
- added C24: 22pF, Capacitor_SMD:C_0603_1608Metric, F.Cu at (108.5, 70.0)
- added C25: 22pF, Capacitor_SMD:C_0603_1608Metric, F.Cu at (116.2, 67.2)
- added C26: 2.2uF, Capacitor_SMD:C_0603_1608Metric, F.Cu at (116.2, 74.2)
- added C27: 100nF, Capacitor_SMD:C_0603_1608Metric, F.Cu at (102.8, 97.5)
- added C28: 100nF, Capacitor_SMD:C_0603_1608Metric, F.Cu at (102.8, 100.0)
- added C29: 100nF, Capacitor_SMD:C_0603_1608Metric, F.Cu at (102.8, 102.5)
- added C3: 10uF, Capacitor_SMD:C_1210_3225Metric, F.Cu at (82.5, 84.2)
- added C30: 100nF, Capacitor_SMD:C_0603_1608Metric, F.Cu at (102.8, 105.0)
- added C31: 100nF, Capacitor_SMD:C_0603_1608Metric, F.Cu at (102.8, 107.5)
- added C32: 100nF, Capacitor_SMD:C_0603_1608Metric, F.Cu at (102.8, 110.0)
- added C33: 100nF, Capacitor_SMD:C_0603_1608Metric, F.Cu at (153.9, 96.2)
- added C34: 100nF, Capacitor_SMD:C_0603_1608Metric, F.Cu at (153.9, 98.7)
- added C4: 10uF, Capacitor_SMD:C_1210_3225Metric, F.Cu at (78.0, 84.2)
- added C5: 100nF, Capacitor_SMD:C_0805_2012Metric, F.Cu at (85.8, 84.2)
- added C6: 100nF, Capacitor_SMD:C_0805_2012Metric, F.Cu at (89.2, 81.0)
- added C7: 10uF, Capacitor_SMD:C_1210_3225Metric, F.Cu at (89.0, 92.8)
- added C8: 10uF, Capacitor_SMD:C_1210_3225Metric, F.Cu at (89.0, 97.2)
- added C9: 2.2uF, Capacitor_SMD:C_0603_1608Metric, F.Cu at (98.5, 81.8)
- added CMC1: PSMCAQ1050-801P, Inductor_SMD:L_CommonModeChoke_Wuerth_WE-SL5, F.Cu at (107.5, 57.5)
- added CMC2: DLW43SH101XK2L, Inductor_SMD:L_CommonModeChoke_Murata_DLW5BTMxxxSQ2x_5x5mm, F.Cu at (118.0, 95.7)
- added CMC3: DLW43SH101XK2L, Inductor_SMD:L_CommonModeChoke_Murata_DLW5BTMxxxSQ2x_5x5mm, F.Cu at (125.0, 95.7)
- added D1: SMAJ18A, Diode_SMD:D_SMA, F.Cu at (90.5, 67.5)
- added D2: 1N5819W1, Diode_SMD:D_SOD-123, F.Cu at (113.8, 86.5)
- added ESD1: CDSOT23-SM712, Package_TO_SOT_SMD:SOT-23-3, F.Cu at (98.2, 98.6)
- added ESD3: CDSOT23-SM712, Package_TO_SOT_SMD:SOT-23-3, F.Cu at (98.2, 107.9)
- added F1: 2.6A PPTC, Fuse:Fuse_1812_4532Metric, F.Cu at (198.5, 125.4)
- added FB1: 200R/100MHz 500mA, Inductor_SMD:L_0805_2012Metric, F.Cu at (113.7, 83.5)
- added FB2: 200R/100MHz 500mA, Inductor_SMD:L_0805_2012Metric, F.Cu at (97.9, 116.1)
- added FB3: 200R/100MHz 500mA, Inductor_SMD:L_0805_2012Metric, F.Cu at (97.9, 118.8)
- added J1: SM10B-ULHK-1TA1-ETB_HF_, SMB10:SM10B-ULHK-1TA1-ETB_HF, F.Cu at (78.2, 60.0)
- added J2: Conn_01x02, Connector_JST:JST_XH_S2B-XH-A_1x02_P2.50mm_Horizontal, F.Cu at (168.3, 85.9)
- added J3: Conn_01x02, Connector_JST:JST_XH_S2B-XH-A_1x02_P2.50mm_Horizontal, F.Cu at (168.3, 76.5)
- added J4: Conn_01x02, Connector_JST:JST_XH_S2B-XH-A_1x02_P2.50mm_Horizontal, F.Cu at (168.3, 67.0)
- added J6: Conn_01x02, Connector_JST:JST_XH_S2B-XH-A_1x02_P2.50mm_Horizontal, F.Cu at (168.3, 57.5)
- added J7: FTSH-107-01-L-DV-K-A, FTSH:SAMTEC_FTSH-107-01-L-DV-K-A, F.Cu at (125.2, 57.0)
- added L1: 33uH, Inductor_SMD:L_TDK_SLF10145, F.Cu at (94.5, 57.0)
- added L2: 4.7uH, Inductor_SMD:L_0603_1608Metric, F.Cu at (85.2, 88.0)
- added R1: 54.9K, Resistor_SMD:R_0805_2012Metric, F.Cu at (90.5, 88.2)
- added R10: 60.4, Resistor_SMD:R_0805_2012Metric, F.Cu at (107.0, 103.6)
- added R11: 60.4, Resistor_SMD:R_0805_2012Metric, F.Cu at (107.0, 106.5)
- added R12: 10K, Resistor_SMD:R_0805_2012Metric, F.Cu at (158.1, 96.4)
- added R13: 100, Resistor_SMD:R_0603_1608Metric, F.Cu at (127.0, 62.0)
- added R14: 0, Resistor_SMD:R_0603_1608Metric, F.Cu at (143.4, 69.5)
- added R15: 0, Resistor_SMD:R_0603_1608Metric, F.Cu at (143.4, 71.5)
- added R16: 100, Resistor_SMD:R_0603_1608Metric, F.Cu at (143.5, 67.5)
- added R17: 100, Resistor_SMD:R_0603_1608Metric, F.Cu at (135.0, 62.8)
- added R18: 100, Resistor_SMD:R_0603_1608Metric, F.Cu at (130.7, 63.5)
- added R19: 100, Resistor_SMD:R_0603_1608Metric, F.Cu at (119.2, 63.8)
- added R2: 10K, Resistor_SMD:R_0805_2012Metric, F.Cu at (87.8, 88.2)
- added R3: 10K, Resistor_SMD:R_0805_2012Metric, F.Cu at (100.8, 84.0)
- added R4: 47, Resistor_SMD:R_0603_1608Metric, F.Cu at (117.4, 83.5)
- added R5: 0, Resistor_SMD:R_0603_1608Metric, F.Cu at (111.2, 72.5)
- added R6: 0, Resistor_SMD:R_0603_1608Metric, F.Cu at (115.4, 64.2)
- added R7: 10K, Resistor_SMD:R_0805_2012Metric, F.Cu at (112.2, 77.2)
- added R8: 60.4, Resistor_SMD:R_0805_2012Metric, F.Cu at (107.0, 97.7)
- added R9: 60.4, Resistor_SMD:R_0805_2012Metric, F.Cu at (107.0, 100.6)
- added SB1: TERM, Jumper:SolderJumper-3_P1.3mm_Open_RoundedPad1.0x1.5mm, F.Cu at (103.6, 113.0)
- added SB2: TERM, Jumper:SolderJumper-3_P1.3mm_Open_RoundedPad1.0x1.5mm, F.Cu at (103.6, 116.9)
- added U2: TLV75733PDBV, Package_TO_SOT_SMD:SOT-23-5, F.Cu at (98.7, 78.4)
- added U3: ISO1050DUB, Package_SO:SOP-8_6.62x9.15mm_P2.54mm, F.Cu at (146.8, 60.0)
- added U4: ISO1050DUB, Package_SO:SOP-8_6.62x9.15mm_P2.54mm, F.Cu at (162.8, 113.2)
- added U5: CA-IS3740HN, Package_SO:SOIC-16_3.9x9.9mm_P1.27mm, F.Cu at (190.8, 128.8)
- added Ue1: TPS562200, Package_TO_SOT_SMD:SOT-23-6, F.Cu at (89.2, 84.2)
- added X1: ASE-16.00MHz, Oscillator:Oscillator_SMD_Abracon_ASE-4Pin_3.2x2.5mm, F.Cu at (117.0, 77.3)
- added Y2: 32.768kHZ, Crystal:Crystal_SMD_3215-2Pin_3.2x1.5mm, F.Cu at (112.0, 67.2)
- moved U1 38.7 mm to (129.0, 73.5)
Connections:
- U1 pad 10: Net-(U1-VSS-Pad10) -> GND
- U1 pad 100: unconnected-(U1-VDD-Pad100) -> +3.3V
- U1 pad 11: unconnected-(U1-VDD-Pad11) -> +3.3V
- U1 pad 12: unconnected-(U1-PH0-Pad12) -> HSE_IN
- U1 pad 14: unconnected-(U1-NRST-Pad14) -> NRST
- U1 pad 19: unconnected-(U1-VSSA-Pad19) -> GND
- U1 pad 20: unconnected-(U1-VREF+-Pad20) -> VREF
- U1 pad 21: unconnected-(U1-VDDA-Pad21) -> VDDA
- U1 pad 26: Net-(U1-VSS-Pad10) -> GND
- U1 pad 27: unconnected-(U1-VDD-Pad27) -> +3.3V
- U1 pad 39: unconnected-(U1-PE9-Pad39) -> RGB_CH_1
- U1 pad 41: unconnected-(U1-PE11-Pad41) -> RGB_CH_2
- U1 pad 43: unconnected-(U1-PE13-Pad43) -> RGB_CH_3
- U1 pad 44: unconnected-(U1-PE14-Pad44) -> RGB_CH_4
- U1 pad 48: unconnected-(U1-VCAP-Pad48) -> Net-(C12-Pad2)
- U1 pad 49: Net-(U1-VSS-Pad10) -> GND
- U1 pad 50: unconnected-(U1-VDD-Pad50) -> +3.3V
- U1 pad 6: unconnected-(U1-VBAT-Pad6) -> +3.3V
- U1 pad 70: unconnected-(U1-PA11-Pad70) -> UART4_RX
- U1 pad 71: unconnected-(U1-PA12-Pad71) -> UART4_TX
- U1 pad 72: unconnected-(U1-PA13-Pad72) -> SWDIO
- U1 pad 73: unconnected-(U1-VCAP-Pad73) -> Net-(C13-Pad2)
- U1 pad 74: Net-(U1-VSS-Pad10) -> GND
- U1 pad 75: unconnected-(U1-VDD-Pad75) -> +3.3V
- U1 pad 76: unconnected-(U1-PA14-Pad76) -> SWCLK
- U1 pad 8: unconnected-(U1-PC14-Pad8) -> LSE_OSC_IN
- U1 pad 89: unconnected-(U1-PB3-Pad89) -> SWO
- U1 pad 9: unconnected-(U1-PC15-Pad9) -> LSE_OSC_OUT
- U1 pad 91: unconnected-(U1-PB5-Pad91) -> CAN_COMM_RX
- U1 pad 92: unconnected-(U1-PB6-Pad92) -> CAN_COMM_TX
- U1 pad 95: unconnected-(U1-PB8-Pad95) -> CAN_CRIT_RX
- U1 pad 96: unconnected-(U1-PB9-Pad96) -> CAN_CRIT_TX
- U1 pad 99: Net-(U1-VSS-Pad10) -> GND
Other:
- copper layers 2 -> 4
