File: PionController/PionController.kicad_pcb (KiCad board)
At the start: 2 copper layers, 1 part, among them U1 STM32H743VITx

Commit message: Schematic_ready
Parts:
- added C1: 10uF, Capacitor_SMD:C_1210_3225Metric, F.Cu at (138.8, 52.5)
- added C11: 10uF, Capacitor_SMD:C_1210_3225Metric, F.Cu at (138.8, 78.0)
- added C12: 2.2uF, Capacitor_SMD:C_0603_1608Metric, F.Cu at (181.1, 77.6)
- added C13: 2.2uF, Capacitor_SMD:C_0603_1608Metric, F.Cu at (181.1, 80.2)
- added C14: 100nF, Capacitor_SMD:C_0603_1608Metric, F.Cu at (181.1, 82.7)
- added C15: 100nF, Capacitor_SMD:C_0603_1608Metric, F.Cu at (181.1, 85.2)
- added C16: 100nF, Capacitor_SMD:C_0603_1608Metric, F.Cu at (181.1, 87.7)
- added C17: 100nF, Capacitor_SMD:C_0603_1608Metric, F.Cu at (181.1, 90.2)
- added C18: 100nF, Capacitor_SMD:C_0603_1608Metric, F.Cu at (185.2, 77.6)
- added C19: 100nF, Capacitor_SMD:C_0603_1608Metric, F.Cu at (185.2, 80.2)
- added C2: 10uF, Capacitor_SMD:C_1210_3225Metric, F.Cu at (138.8, 56.8)
- added C20: 2.2uF, Capacitor_SMD:C_0603_1608Metric, F.Cu at (185.2, 82.7)
- added C21: 2.2uF, Capacitor_SMD:C_0603_1608Metric, F.Cu at (185.2, 85.2)
- added C22: 100nF, Capacitor_SMD:C_0603_1608Metric, F.Cu at (185.2, 87.7)
- added C23: 100nF, Capacitor_SMD:C_0603_1608Metric, F.Cu at (185.2, 90.2)
- added C24: 22pF, Capacitor_SMD:C_0603_1608Metric, F.Cu at (189.2, 77.6)
- added C25: 22pF, Capacitor_SMD:C_0603_1608Metric, F.Cu at (189.2, 80.2)
- added C26: 2.2uF, Capacitor_SMD:C_0603_1608Metric, F.Cu at (189.2, 82.7)
- added C27: 100nF, Capacitor_SMD:C_0603_1608Metric, F.Cu at (180.8, 51.6)
- added C28: 100nF, Capacitor_SMD:C_0603_1608Metric, F.Cu at (180.8, 54.2)
- added C29: 100nF, Capacitor_SMD:C_0603_1608Metric, F.Cu at (180.8, 56.7)
- added C3: 10uF, Capacitor_SMD:C_1210_3225Metric, F.Cu at (138.8, 61.0)
- added C30: 100nF, Capacitor_SMD:C_0603_1608Metric, F.Cu at (180.8, 59.2)
- added C31: 100nF, Capacitor_SMD:C_0603_1608Metric, F.Cu at (180.8, 61.7)
- added C32: 100nF, Capacitor_SMD:C_0603_1608Metric, F.Cu at (180.8, 64.2)
- added C4: 10uF, Capacitor_SMD:C_1210_3225Metric, F.Cu at (138.8, 65.3)
- added C5: 100nF, Capacitor_SMD:C_0805_2012Metric, F.Cu at (152.0, 74.3)
- added C6: 100nF, Capacitor_SMD:C_0805_2012Metric, F.Cu at (152.0, 77.3)
- added C7: 10uF, Capacitor_SMD:C_1210_3225Metric, F.Cu at (138.8, 69.5)
- added C8: 10uF, Capacitor_SMD:C_1210_3225Metric, F.Cu at (138.8, 73.8)
- added CMC1: PSMCAQ1050-801P, Inductor_SMD:L_CommonModeChoke_Wuerth_WE-SL5, F.Cu at (147.6, 67.6)
- added D1: SMAJ18A, Diode_SMD:D_SMA, F.Cu at (145.7, 75.1)
- added D2: 1N5819W1, Diode_SMD:D_SOD-123, F.Cu at (182.1, 93.1)
- added ESD1: CDSOT23-SM712, Package_TO_SOT_SMD:SOT-23-3, F.Cu at (176.2, 52.8)
- added ESD2: CDSOT23-SM712, Package_TO_SOT_SMD:SOT-23-3, F.Cu at (176.2, 57.4)
- added ESD3: CDSOT23-SM712, Package_TO_SOT_SMD:SOT-23-3, F.Cu at (176.2, 62.0)
- added ESD4: CDSOT23-SM712, Package_TO_SOT_SMD:SOT-23-3, F.Cu at (176.2, 66.7)
- added F1: 2.6A PPTC, Fuse:Fuse_1812_4532Metric, F.Cu at (147.9, 84.6)
- added FB1: 200R/100MHz 500mA, Inductor_SMD:L_0805_2012Metric, F.Cu at (162.9, 96.3)
- added FB2: 200R/100MHz 500mA, Inductor_SMD:L_0805_2012Metric, F.Cu at (175.9, 70.3)
- added FB3: 200R/100MHz 500mA, Inductor_SMD:L_0805_2012Metric, F.Cu at (175.9, 73.0)
- added L1: 33uH, Inductor_SMD:L_TDK_SLF10145, F.Cu at (147.8, 56.5)
- added L2: 4.7uH, Inductor_SMD:L_0603_1608Metric, F.Cu at (156.2, 74.1)
- added R1: 54.9K, Resistor_SMD:R_0805_2012Metric, F.Cu at (156.0, 51.9)
- added R10: 60.4, Resistor_SMD:R_0805_2012Metric, F.Cu at (185.0, 57.8)
- added R11: 60.4, Resistor_SMD:R_0805_2012Metric, F.Cu at (185.0, 60.7)
- added R2: 10K, Resistor_SMD:R_0805_2012Metric, F.Cu at (156.0, 54.8)
- added R3: 10K, Resistor_SMD:R_0805_2012Metric, F.Cu at (156.0, 57.8)
- added R5: 0, Resistor_SMD:R_0603_1608Metric, F.Cu at (189.2, 85.2)
- added R6: 0, Resistor_SMD:R_0603_1608Metric, F.Cu at (189.2, 87.7)
- added R7: 10K, Resistor_SMD:R_0805_2012Metric, F.Cu at (167.4, 96.4)
- added R8: 60.4, Resistor_SMD:R_0805_2012Metric, F.Cu at (185.0, 51.9)
- added R9: 60.4, Resistor_SMD:R_0805_2012Metric, F.Cu at (185.0, 54.8)
- added SB1: TERM, Jumper:SolderJumper-3_P1.3mm_Open_RoundedPad1.0x1.5mm, F.Cu at (181.6, 67.2)
- added SB2: TERM, Jumper:SolderJumper-3_P1.3mm_Open_RoundedPad1.0x1.5mm, F.Cu at (181.6, 71.1)
- added U2: TLV75733PDBV, Package_TO_SOT_SMD:SOT-23-5, F.Cu at (156.1, 64.7)
- added U3: ISO1050DUB, Package_SO:SOP-8_6.62x9.15mm_P2.54mm, F.Cu at (167.1, 55.8)
- added U4: ISO1050DUB, Package_SO:SOP-8_6.62x9.15mm_P2.54mm, F.Cu at (167.1, 66.6)
- added U5: CA-IS3740HN, Package_SO:SOIC-16_3.9x9.9mm_P1.27mm, F.Cu at (140.2, 88.0)
- added Ue1: TPS562200, Package_TO_SOT_SMD:SOT-23-6, F.Cu at (156.1, 69.3)
- added X1: ASE-16.00MHz, Oscillator:Oscillator_SMD_Abracon_ASE-4Pin_3.2x2.5mm, F.Cu at (187.4, 93.7)
- added Y2: 32.768kHZ, Crystal:Crystal_SMD_3215-2Pin_3.2x1.5mm, F.Cu at (181.7, 96.5)
- moved U1 70.9 mm to (169.9, 85.6)
Connections:
- U1 pad 10: Net-(U1-VSS-Pad10) -> GND
- U1 pad 100: unconnected-(U1-VDD-Pad100) -> +3.3V
- U1 pad 11: unconnected-(U1-VDD-Pad11) -> +3.3V
- U1 pad 12: unconnected-(U1-PH0-Pad12) -> HSE_IN
- U1 pad 19: unconnected-(U1-VSSA-Pad19) -> GND
- U1 pad 20: unconnected-(U1-VREF+-Pad20) -> VREF
- U1 pad 21: unconnected-(U1-VDDA-Pad21) -> VDDA
- U1 pad 26: Net-(U1-VSS-Pad10) -> GND
- U1 pad 27: unconnected-(U1-VDD-Pad27) -> +3.3V
- U1 pad 48: unconnected-(U1-VCAP-Pad48) -> Net-(C12-Pad2)
- U1 pad 49: Net-(U1-VSS-Pad10) -> GND
- U1 pad 50: unconnected-(U1-VDD-Pad50) -> +3.3V
- U1 pad 6: unconnected-(U1-VBAT-Pad6) -> +3.3V
- U1 pad 73: unconnected-(U1-VCAP-Pad73) -> Net-(C13-Pad2)
- U1 pad 74: Net-(U1-VSS-Pad10) -> GND
- U1 pad 75: unconnected-(U1-VDD-Pad75) -> +3.3V
- U1 pad 8: unconnected-(U1-PC14-Pad8) -> LSE_OSC_IN
- U1 pad 9: unconnected-(U1-PC15-Pad9) -> LSE_OSC_OUT
- U1 pad 91: unconnected-(U1-PB5-Pad91) -> CAN_COMM_RX
- U1 pad 92: unconnected-(U1-PB6-Pad92) -> CAN_COMM_TX
- U1 pad 95: unconnected-(U1-PB8-Pad95) -> CAN_CRIT_RX
- U1 pad 96: unconnected-(U1-PB9-Pad96) -> CAN_CRIT_TX
- U1 pad 99: Net-(U1-VSS-Pad10) -> GND

Commit message: fix
Parts:
- removed ESD2, ESD4: CDSOT23-SM712, Package_TO_SOT_SMD:SOT-23-3
- added C10: 2.2uF, Capacitor_SMD:C_0603_1608Metric, F.Cu at (102.0, 80.8)
- added C33: 100nF, Capacitor_SMD:C_0603_1608Metric, F.Cu at (153.9, 96.2)
- added C34: 100nF, Capacitor_SMD:C_0603_1608Metric, F.Cu at (153.9, 98.7)
- added C9: 2.2uF, Capacitor_SMD:C_0603_1608Metric, F.Cu at (98.5, 81.8)
- added CMC2: DLW43SH101XK2L, Inductor_SMD:L_CommonModeChoke_Murata_DLW5BTMxxxSQ2x_5x5mm, F.Cu at (96.2, 91.5)
- added CMC3: DLW43SH101XK2L, Inductor_SMD:L_CommonModeChoke_Murata_DLW5BTMxxxSQ2x_5x5mm, F.Cu at (103.2, 91.5)
- added J1: SM10B-ULHK-1TA1-ETB_HF_, SMB10:SM10B-ULHK-1TA1-ETB_HF, F.Cu at (78.2, 60.0)
- added J2: Conn_01x02, Connector_JST:JST_XH_S2B-XH-A_1x02_P2.50mm_Horizontal, F.Cu at (168.3, 85.9)
- added J3: Conn_01x02, Connector_JST:JST_XH_S2B-XH-A_1x02_P2.50mm_Horizontal, F.Cu at (168.3, 76.5)
- added J4: Conn_01x02, Connector_JST:JST_XH_S2B-XH-A_1x02_P2.50mm_Horizontal, F.Cu at (168.3, 67.0)
- added J6: Conn_01x02, Connector_JST:JST_XH_S2B-XH-A_1x02_P2.50mm_Horizontal, F.Cu at (168.3, 57.5)
- added J7: FTSH-107-01-L-DV-K-A, FTSH:SAMTEC_FTSH-107-01-L-DV-K-A, F.Cu at (125.2, 57.0)
- added R12: 10K, Resistor_SMD:R_0805_2012Metric, F.Cu at (158.1, 96.4)
- added R13: 100, Resistor_SMD:R_0603_1608Metric, F.Cu at (127.0, 62.0)
- added R14: 0, Resistor_SMD:R_0603_1608Metric, F.Cu at (143.4, 69.5)
- added R15: 0, Resistor_SMD:R_0603_1608Metric, F.Cu at (143.4, 71.5)
- added R16: 100, Resistor_SMD:R_0603_1608Metric, F.Cu at (143.5, 67.5)
- added R17: 100, Resistor_SMD:R_0603_1608Metric, F.Cu at (135.0, 62.8)
- added R18: 100, Resistor_SMD:R_0603_1608Metric, F.Cu at (130.7, 63.5)
- added R19: 100, Resistor_SMD:R_0603_1608Metric, F.Cu at (119.2, 63.8)
- added R4: 47, Resistor_SMD:R_0603_1608Metric, F.Cu at (117.4, 83.5)
- moved U4 94.2 mm to (88.5, 118.5), turned to 180 degrees
- moved U3 93.1 mm to (88.8, 106.0)
- moved C27 90.4 mm to (102.8, 97.5)
- moved C28 90.4 mm to (102.8, 100.0)
- moved C29 90.4 mm to (102.8, 102.5)
- moved C30 90.4 mm to (102.8, 105.0)
- moved C31 90.4 mm to (102.8, 107.5)
- moved C32 90.4 mm to (102.8, 110.0)
- moved ESD1 90.4 mm to (98.2, 98.6)
- moved ESD3 90.4 mm to (98.2, 107.9)
- moved FB2 90.4 mm to (97.9, 116.1)
- moved FB3 90.4 mm to (97.9, 118.8)
- moved R10 90.4 mm to (107.0, 103.6)
- moved R11 90.4 mm to (107.0, 106.5)
- moved R8 90.4 mm to (107.0, 97.7)
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Connections:
- U1 pad 14: unconnected-(U1-NRST-Pad14) -> NRST
- U1 pad 39: unconnected-(U1-PE9-Pad39) -> RGB_CH_1
- U1 pad 41: unconnected-(U1-PE11-Pad41) -> RGB_CH_2
- U1 pad 43: unconnected-(U1-PE13-Pad43) -> RGB_CH_3
- U1 pad 44: unconnected-(U1-PE14-Pad44) -> RGB_CH_4
- U1 pad 70: unconnected-(U1-PA11-Pad70) -> UART4_RX
- U1 pad 71: unconnected-(U1-PA12-Pad71) -> UART4_TX
- U1 pad 72: unconnected-(U1-PA13-Pad72) -> SWDIO
- U1 pad 76: unconnected-(U1-PA14-Pad76) -> SWCLK
- U1 pad 89: unconnected-(U1-PB3-Pad89) -> SWO
- U5 pad 10: +5V -> Net-(U5-EN)
- U5 pad 11: unconnected-(U5-OUTD-Pad11) -> Net-(J6-Pin_2)
- U5 pad 12: unconnected-(U5-OUTC-Pad12) -> Net-(J4-Pin_2)
- U5 pad 13: unconnected-(U5-OUTB-Pad13) -> Net-(J3-Pin_2)
- U5 pad 14: unconnected-(U5-OUTA-Pad14) -> Net-(J2-Pin_2)
- U5 pad 3: unconnected-(U5-INA-Pad3) -> RGB_CH_1
- U5 pad 4: unconnected-(U5-INB-Pad4) -> RGB_CH_2
- U5 pad 5: unconnected-(U5-INC-Pad5) -> RGB_CH_3
- U5 pad 6: unconnected-(U5-IND-Pad6) -> RGB_CH_4
Other:
- copper layers 2 -> 4

Commit message: just messing aroung
Parts:
- SB1: moved to B.Cu
- moved C11 122.3 mm to (229.7, 102.7)
- moved C12 107.9 mm to (179.1, 46.9)
- moved C13 107.9 mm to (179.1, 49.4)
- moved FB2 99.8 mm to (177.9, 56.4)
- moved FB3 99.8 mm to (177.9, 59.1)
- moved C32 88.3 mm to (159.6, 42.5), turned to 90 degrees
- moved F1 88.1 mm to (113.1, 103.8)
- moved C31 84.7 mm to (157.1, 42.5), turned to 90 degrees
- moved J6 81.7 mm to (153.2, 137.8), turned to 0 degrees
- moved C30 81.2 mm to (154.6, 42.5), turned to 90 degrees
- moved J7 77.9 mm to (202.9, 50.5)
- moved C29 77.7 mm to (152.1, 42.5), turned to 90 degrees
- moved SB2 75.1 mm to (154.7, 61.8), turned to 90 degrees
- moved J4 74.9 mm to (143.8, 137.8), turned to 0 degrees
- moved C28 74.1 mm to (149.6, 42.5), turned to 90 degrees
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Routing:
- net +5V: track 0.00 -> 19.3 mm
- net Net-(Ue1-SW): track 0.00 -> 6.64 mm
- net +3.3V: track 0.00 -> 5.14 mm, vias 0 -> 3
- net +12V: track 0.00 -> 2.67 mm
- net Net-(U2-EN): track 0.00 -> 2.02 mm
- net Net-(Ue1-VBST): track 0.00 -> 2.00 mm
- net Net-(Ue1-VFB): track 0.00 -> 1.80 mm
- net GND: track 0.00 -> 0.97 mm, vias 0 -> 1
- added copper zone on F.Cu, net +12V
- added copper zone on F.Cu, net +12V_CAR
- added copper zone on F.Cu, net +3.3V
- added copper zone on In2.Cu, net +3.3V
- added copper zone on F.Cu, net /Connectors/Vbus
- added copper zone on In1.Cu, net GND
- added copper zone on F.Cu, net Net-(C1-Pad1)

Commit message: commit to be happy
Parts:
- SB2: moved to B.Cu
- moved C11 97.9 mm to (133.0, 118.0), turned to 180 degrees
- moved C33 87.4 mm to (128.9, 131.8)
- moved FB2 83.9 mm to (111.9, 108.2), turned to -90 degrees
- moved FB3 80.1 mm to (114.6, 108.2), turned to -90 degrees
- moved R12 78.1 mm to (145.5, 133.3)
- moved J7 76.0 mm to (132.6, 79.5)
- moved C29 69.8 mm to (112.3, 99.8), turned to 180 degrees
- moved C32 65.7 mm to (112.0, 87.8), turned to 180 degrees
- moved C28 59.2 mm to (125.3, 96.5), turned to -90 degrees
- moved C27 55.5 mm to (139.6, 97.5), turned to -90 degrees
- moved C31 51.4 mm to (129.9, 86.2), turned to 0 degrees
- moved SB2 48.2 mm to (115.4, 89.8)
- moved C13 44.3 mm to (144.8, 77.4), turned to -90 degrees
- moved C30 43.3 mm to (126.8, 75.7), turned to -90 degrees
- moved C12 40.9 mm to (159.8, 82.9)
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Routing:
- net GND: track 0.97 -> 54.8 mm, vias 1 -> 20
- net Net-(U4-VCC2): track 0.00 -> 43.8 mm
- net Net-(U3-VCC2): track 0.00 -> 28.9 mm
- net CAN_CRIT_H: track 0.00 -> 12.6 mm
- net CAN_COMM_L: track 0.00 -> 12.3 mm
- net CAN_CRIT_L: track 0.00 -> 12.3 mm
- net CAN_COMM_H: track 0.00 -> 12.2 mm
- net VDDA: track 0.00 -> 11.8 mm
- net CAN_CRIT_RX: track 0.00 -> 11.8 mm
- net Net-(U3-CANH): track 0.00 -> 9.57 mm
- net Net-(U4-CANH): track 0.00 -> 9.21 mm
- net Net-(U3-CANL): track 0.00 -> 8.29 mm
- net HSE_IN: track 0.00 -> 7.79 mm
- net LSE_OSC_OUT: track 0.00 -> 6.80 mm
- net LSE_OSC_IN: track 0.00 -> 6.39 mm
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
Commit message: Version 1
Parts:
- removed C2: 10uF, Capacitor_SMD:C_1210_3225Metric
- removed L1: 33uH, Inductor_SMD:L_TDK_SLF10145
- moved J2 78.8 mm to (175.0, 84.8), turned to 90 degrees
- moved J3 66.0 mm to (175.0, 93.5), turned to 90 degrees
- moved U5 54.8 mm to (165.5, 85.9), turned to 0 degrees
- moved J4 53.3 mm to (175.0, 102.2), turned to 90 degrees
- moved C33 51.2 mm to (163.1, 93.6), turned to 90 degrees
- moved R12 44.4 mm to (165.5, 93.6), turned to -90 degrees
- moved J6 40.6 mm to (174.9, 111.1), turned to 90 degrees
- moved FB2 24.6 mm to (136.3, 111.0)
- moved C30 22.9 mm to (135.6, 96.8), turned to 0 degrees
- moved FB3 17.4 mm to (128.0, 97.3)
- moved C10 15.5 mm to (133.0, 111.7)
- moved C9 15.5 mm to (130.6, 115.2)
- moved C1 15.5 mm to (121.7, 101.8)
- moved C5 15.5 mm to (121.0, 118.7)
- moved CMC1 15.5 mm to (124.9, 109.6)
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Connections:
- net /Connectors/Vbus renamed Net-(F1-Pad1)
- C1 pad 1: Net-(C1-Pad1) -> +12V_CAR
- C18 pad 1: +3.3V -> GND
- C18 pad 2: GND -> +3.3V
- CMC1 pad 2: Net-(C1-Pad1) -> +12V_CAR
- U5 pad 3: RGB_CH_1 -> RGB_CH_4
- U5 pad 4: RGB_CH_2 -> RGB_CH_3
- U5 pad 5: RGB_CH_3 -> RGB_CH_2
- U5 pad 6: RGB_CH_4 -> RGB_CH_1
Routing:
- net +5V: track 21.0 -> 117.6 mm
- net GND: track 54.8 -> 111.1 mm, vias 20 -> 62
- net Net-(J7-Pad13): track 0.00 -> 55.5 mm
- net Net-(U4-VCC2): track 43.8 -> 4.15 mm
- net Net-(J7-Pad04): track 0.00 -> 27.0 mm
- net Net-(J6-Pin_2): track 0.00 -> 26.2 mm
- net +3.3V: track 7.58 -> 33.8 mm, vias 5 -> 18
- net NRST: track 0.00 -> 20.8 mm
- net Net-(U3-VCC2): track 28.9 -> 8.34 mm
- net Net-(J4-Pin_2): track 0.00 -> 19.2 mm
- net Net-(J7-Pad14): track 0.00 -> 17.9 mm, vias 0 -> 2
- net Net-(J7-Pad06): track 0.00 -> 15.3 mm
- net CAN_COMM_RX: track 0.00 -> 13.9 mm
- net SWO: track 0.00 -> 13.4 mm
- net Net-(J7-Pad08): track 0.00 -> 11.8 mm
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- removed copper zone on F.Cu, net Net-(C1-Pad1)

Commit message: Version 1.2
Parts:
- moved J2 1.04 mm to (173.9, 84.9)
- moved J3 1.04 mm to (173.9, 93.6)
- moved J4 1.04 mm to (173.9, 102.3)
- moved J6 1.04 mm to (173.9, 111.2)
- moved U5 0.43 mm to (165.1, 85.9)
Routing:
- net Net-(J7-Pad13): track 55.5 -> 49.3 mm
- net GND: track 111.1 -> 106.7 mm
- net Net-(J7-Pad04): track 27.0 -> 24.9 mm
- net Net-(J7-Pad14): track 17.9 -> 16.3 mm
- net Net-(J7-Pad06): track 15.3 -> 14.2 mm
- net Net-(J7-Pad12): track 10.8 -> 9.69 mm
- net Net-(J7-Pad08): track 11.8 -> 10.9 mm
- net Net-(J4-Pin_2): track 19.2 -> 18.6 mm
- net Net-(J6-Pin_2): track 26.2 -> 25.7 mm
- net Net-(J2-Pin_2): track 7.66 -> 7.08 mm
- net Net-(J3-Pin_2): track 11.4 -> 10.8 mm
